Commit message: Add files via upload

File: hand_description/urdf/hand.urdf (robot description, URDF)
Before this commit: robot None, 7 links, 6 joints
Links:
- removed link idol_pivot_grip
- removed link servo_pivot_grip
- link base_hand: mass None -> 0.059408; geometry collision mesh filename=package://hand_description/meshes/base_tool.stl scale=0.001 0.001 0.001; visual mesh filename=package://hand_description/meshes/base_tool.stl scale=0.001 0.001 0.001
- link idol_gear: mass None -> 0.0052; geometry collision mesh filename=package://hand_description/meshes/idol_gear.stl scale=0.001 0.001 0.001; visual mesh filename=package://hand_description/meshes/idol_gear.stl scale=0.001 0.001 0.001
- link idol_grip: mass None -> 0.013967; geometry collision mesh filename=package://hand_description/meshes/idol_grip.stl scale=0.001 0.001 0.001; visual mesh filename=package://hand_description/meshes/idol_grip.stl scale=0.001 0.001 0.001
- link servo_gear: mass None -> 0.005069; geometry collision mesh filename=package://hand_description/meshes/servo_gear.stl scale=0.001 0.001 0.001; visual mesh filename=package://hand_description/meshes/servo_gear.stl scale=0.001 0.001 0.001
- link servo_grip: mass None -> 0.013967; geometry collision mesh filename=package://hand_description/meshes/servo_grip.stl scale=0.001 0.001 0.001; visual mesh filename=package://hand_description/meshes/servo_grip.stl scale=0.001 0.001 0.001
Joints:
- removed joint idol_pivot_grip_joint
- removed joint servo_pivot_grip_joint
- added joint joint_6: type fixed, parent link_5, child base_hand, origin xyz=0 0 0.041 rpy=0 0 0, axis 1 0 0
