Commit message: Add files via upload

File: hand_description/urdf/gazebo_hand.xacro (robot description, xacro)
@@ -1,4 +1,34 @@
 <?xml version="1.0" ?>
 <robot name="moveo" xmlns:xacro="http://www.ros.org/wiki/xacro" >
+  	<gazebo>
+		<plugin name="idol_grip_joint_mimic_plugin" filename="libroboticsgroup_gazebo_mimic_joint_plugin.so">
+			<joint>idol_grip_joint</joint>
+			<mimicJoint>idol_gear_joint</mimicJoint>
+			<multiplier>-1</multiplier>
+			<offset>0.0</offset>
+			<maxEffort>30.0</maxEffort>
+			<sensitiveness>0.0</sensitiveness>
+		</plugin>
+	</gazebo>
+  	<gazebo>
+		<plugin name="servo_gear_joint_mimic_plugin" filename="libroboticsgroup_gazebo_mimic_joint_plugin.so">
+			<joint>servo_gear_joint</joint>
+			<mimicJoint>idol_gear_joint</mimicJoint>
+			<multiplier>-1</multiplier>
+			<offset>0.0</offset>
+			<maxEffort>30.0</maxEffort>
+			<sensitiveness>0.0</sensitiveness>
+		</plugin>
+	</gazebo>
+  	<gazebo>
+		<plugin name="servo_grip_joint_mimic_plugin" filename="libroboticsgroup_gazebo_mimic_joint_plugin.so">
+			<joint>servo_grip_joint</joint>
+			<mimicJoint>servo_gear_joint</mimicJoint>
+			<multiplier>-1</multiplier>
+			<offset>0.0</offset>
+			<maxEffort>30.0</maxEffort>
+			<sensitiveness>0.0</sensitiveness>
+		</plugin>
+	</gazebo>
     <gazebo reference="base_hand">
         <mu1>0.2</mu1>
@@ -27,3 +57,8 @@
         <selfCollide>true</selfCollide>
     </gazebo>
+	<gazebo>
+		<plugin name="gazebo_ros_control" filename="libgazebo_ros_control.so" >
+		<controlPeriod>0.001</controlPeriod>
+		</plugin>
+	</gazebo>
 </robot>

File: hand_description/urdf/hand.urdf (robot description, URDF)
Before this commit: robot None, 5 links, 5 joints
Links:
- removed link base_hand
- added link hand_base_link, mass 0.059408; collision mesh filename=package://hand_description/meshes/base_tool.stl scale=0.001 0.001 0.001; visual mesh filename=package://hand_description/meshes/base_tool.stl scale=0.001 0.001 0.001
Joints:
- removed joint joint_6
- joint idol_gear_joint: parent base_hand -> hand_base_link
- joint idol_grip_joint: limit (none) -> lower=-0.5 upper=1.15 effort=30 velocity=1.5; type continuous -> revolute
- joint servo_gear_joint: parent base_hand -> hand_base_link
- joint servo_grip_joint: limit (none) -> lower=-0.5 upper=1.15 effort=100 velocity=2

File: moveo_description/urdf/gazebo_moveo.xacro (robot description, xacro)
@@ -2,6 +2,11 @@
 <robot name="moveo" xmlns:xacro="http://www.ros.org/wiki/xacro" >
     <gazebo>
-        <plugin name="gazebo_ros_control" filename="libgazebo_ros_control.so">
-            <robotNamespace>/moveo</robotNamespace>
+        <plugin name="gazebo_ros_control" filename="libgazebo_ros_control.so" >
+        <!--robotNamespace>wam</robotNamespace-->
+        <!-- Custom plugin -->
+        <!-- robotSimType>wam_gazebo_ros_control/WamRobotHWSim</robotSimType -->
+        <!-- Default plugin -->
+        <!-- robotSimType>gazebo_ros_control/DefaultRobotHWSim</robotSimType -->
+        <controlPeriod>0.001</controlPeriod>
         </plugin>
     </gazebo>
