Commit message: Add files via upload

File: moveo_description/urdf/moveo.urdf (robot description, URDF)
Before this commit: robot moveo, 7 links, 6 joints
Links:
- added link link_6; visual box size=0.01 0.01 0.01
Joints:
- removed joint fixed
- added joint joint_6: type fixed, parent link_5, child link_6, origin xyz=0.1 0 0 rpy=0 0 0
- added joint world_joint: type fixed, parent world, child base_link, origin xyz=0.0 0.0 0.0 rpy=0.0 0.0 0.0
- joint joint_1: limit lower=-1.570796 upper=1.570796 effort=100 velocity=2 -> lower=-1.570796 upper=1.570796 effort=28.0 velocity=3.2; origin xyz=0 0 0.14695 rpy=0 0 0 -> xyz=0 0 0.14695 rpy=0 0 ${pi/2}
- joint joint_2: axis 1 0 0 -> 0 0 1; limit lower=-1.570796 upper=1.570796 effort=100 velocity=2 -> lower=-1.570796 upper=1.570796 effort=28.0 velocity=3.2; origin xyz=0.0015 0 0.1655 rpy=0 0 0 -> xyz=0 0 0.1655 rpy=${pi/2} ${-pi/2} 0
- joint joint_3: axis 1 0 0 -> 0 0 1; limit lower=-1.570796 upper=1.570796 effort=100 velocity=2 -> lower=-1.570796 upper=1.570796 effort=28.0 velocity=3.2; origin xyz=0.002 0 0.22112 rpy=0 0 0 -> xyz=0.22112 0 0 rpy=0 0 0
- joint joint_4: axis 0 0 1 -> 1 0 0; limit lower=-1.570796 upper=1.570796 effort=100 velocity=2 -> lower=-1.570796 upper=1.570796 effort=28.0 velocity=3.2; origin xyz=0 0 0.12762 rpy=0 0 0 -> xyz=0.12762 0 0 rpy=0 0 0
- joint joint_5: axis 1 0 0 -> 0 0 1; limit lower=-1.570796 upper=1.570796 effort=100 velocity=2 -> lower=-1.570796 upper=1.570796 effort=28.0 velocity=3.2; origin xyz=0 0 0.095 rpy=0 0 0 -> xyz=0.095 0 0 rpy=0 0 0
